File: kicad/supply_power/supply_power.kicad_pcb (KiCad board)
At the start: 4 copper layers, 170 x 74.5 mm, 247 parts, among them J101 USB_C_Receptacle_USB2.0_16P, J161 DC IN wires, J951 B2B to supply_control, Q101 CSD18540Q5B, Q102 CSD18540Q5B, Q161 ISC030N10NM6, Q162 ISC030N10NM6, Q201 2N7002, Q202 CSD18531Q5A, Q203 CSD18531Q5A, Q301 BC857, Q302 2N7002, Q401 BSC040N10NS5, Q402 BSC040N10NS5, Q403 BSC040N10NS5, Q404 2N7002, Q405 2N7002, U101 AP33772S, U102 LM74800, U161 LM74800, U181 INA228, U201 LTC7803, U202 INA240A3PW, U301 ADA4522-2, U302 LMV331, U401 INA228, U402 LMV331, U403 LMV331, U404 UCC27511ADBV, U405 VOM1271, U541 LM5164DDA, U542 LP2985-5.0

Commit message: added encoder model
Parts:
- added D162: BZT52C12, Diode_SMD:D_SOD-123, F.Cu at (148.4, 106.4)
- added Q163: 2N7002, Package_TO_SOT_SMD:SOT-23, F.Cu at (88.5, 118.4)
- added Q164: 2N7002, Package_TO_SOT_SMD:SOT-23, F.Cu at (88.5, 114.5)
- added R165: 1M, Resistor_SMD:R_0603_1608Metric, F.Cu at (91.3, 113.6)
- added R166: 100k, Resistor_SMD:R_0603_1608Metric, F.Cu at (88.7, 111.5)
- added TP161: TestPoint, TestPoint:TestPoint_Pad_D1.0mm, F.Cu at (91.5, 110.8)
- moved C313 60.2 mm to (231.5, 126.7), turned to 0 degrees
- moved R315 57.9 mm to (228.2, 126.9), turned to 180 degrees
- moved R314 56.6 mm to (230.7, 124.1), turned to -90 degrees
- moved C311 56.6 mm to (219.8, 101.0)
- moved R310 56.6 mm to (219.7, 99.2)
- moved R311 56.6 mm to (219.7, 97.5)
- moved R312 56.6 mm to (217.2, 99.2)
- moved C312 56.6 mm to (219.7, 95.7)
- moved D303 56.6 mm to (218.9, 92.7)
- moved R313 56.6 mm to (216.4, 96.7)
- moved U302 54.1 mm to (228.0, 123.8), turned to 90 degrees
- moved C314 51.6 mm to (225.3, 123.4), turned to -90 degrees
- moved R316 50.6 mm to (228.2, 120.6), turned to 0 degrees
- moved H906 27.6 mm to (153.7, 111.5), turned to -90 degrees
- moved F401 26.0 mm to (189.4, 82.5), turned to 90 degrees
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Connections:
- J951 pad 22: GND -> DCIN_ON
Routing:
- net USBIN_MID: track 17.5 -> 9.42 mm, vias 2 -> 0
- net N$14: track 4.12 -> 0.04 mm
