File: kicad/supply_control/supply_control.kicad_pcb (KiCad board)
At the start: 4 copper layers, 110 x 74.5 mm, 75 parts, among them J601 USB_C_Receptacle_USB2.0_16P, J701 SWD, J702 UART, J703 UI ribbon, J971 B2B to supply_power, SW701 RESET, SW702 BOOT, U501 LMR38010, U601 USBLC6-2SC6, U602 ADUM3160, U701 STM32G474RETx

Commit message: added encoder model
Parts:
- added C509: 10n, Capacitor_SMD:C_0603_1608Metric, F.Cu at (126.4, 111.8)
- added J501: POWER rocker, Connector_JST:JST_XH_B2B-XH-A_1x02_P2.50mm_Vertical, F.Cu at (122.4, 112.8)
- added R505: 4.7k, Resistor_SMD:R_1206_3216Metric, F.Cu at (131.4, 123.5)
- added R506: 47k, Resistor_SMD:R_0603_1608Metric, F.Cu at (124.4, 120.1)
- added TP502: TestPoint, TestPoint:TestPoint_Pad_D1.0mm, F.Cu at (127.7, 123.3)
- moved C503 6.47 mm to (126.9, 119.3), turned to 180 degrees
- moved D503 6.12 mm to (129.2, 109.5)
- moved C506 4.85 mm to (136.8, 124.2), turned to -90 degrees
- moved TP501 4.17 mm to (139.1, 123.5)
- moved R504 3.76 mm to (140.6, 120.6)
- moved D504 3.54 mm to (140.6, 117.1)
- moved C501 3.51 mm to (127.2, 115.8), turned to 90 degrees
- moved R501 3.17 mm to (127.4, 121.1)
- moved U501 3.17 mm to (132.4, 116.4)
- moved R502 3.17 mm to (134.8, 120.9)
- moved R503 3.17 mm to (137.9, 119.1)
- moved C505 3.17 mm to (137.5, 121.2)
- moved C504 3.17 mm to (137.3, 116.5)
- moved C502 3.17 mm to (131.4, 120.8)
- moved L501 1.69 mm to (134.6, 109.7)
Connections:
- J703 pad 18: PWR_BTN -> LCD_BL
- J971 pad 21: GND -> DCIN_ON
- U501 pad 2: LOGIC_IN -> LOG_EN
- U701 pad 2: PWR_BTN -> (no net)
- U701 pad 30: (no net) -> LCD_BL
- U701 pad 57: (no net) -> DCIN_ON

Commit message: Checkpoint before ui routing
Parts:
- moved J703 6.50 mm to (208.6, 82.3)
Changed lines of the file:
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@@
 	(footprint "Connector_PinHeader_1.27mm:PinHeader_2x10_P1.27mm_Vertical"
 		(layer "F.Cu")
-		(at 202.115 82.285)
+		(at 208.615 82.285)
 		(descr "Through hole straight pin header, 2x10, 1.27mm pitch, double rows")
 		(tags "Through hole pin header THT 2x10 1.27mm double row")
@@
 		(locked yes)
 		(layer "B.Cu")
-		(name "floorplan: C223 on the power board below (tall)")
+		(name "floorplan: C228 on the power board below (tall)")
 		(hatch edge 0.5)
 		(connect_pads
@@
 		(polygon
 			(pts
-				(xy 190.706249 81.207498) (xy 203.29375 81.207498) (xy 203.29375 93.792502) (xy 190.706249 93.792502)
+				(xy 201.555 80.555) (xy 217.245 80.555) (xy 217.245 93.445) (xy 201.555 93.445)
 			)
 		)
@@
 		(locked yes)
 		(layer "B.Cu")
-		(name "floorplan: C228 on the power board below (tall)")
+		(name "floorplan: C223 on the power board below (tall)")
 		(hatch edge 0.5)
 		(connect_pads
@@
 		(polygon
 			(pts
-				(xy 201.555 80.555) (xy 217.245 80.555) (xy 217.245 93.445) (xy 201.555 93.445)
+				(xy 190.706249 81.207498) (xy 203.29375 81.207498) (xy 203.29375 93.792502) (xy 190.706249 93.792502)
 			)
 		)
@@
 		)
 	)
-	(group "place:B2B decoupling"
-		(members "19df6b39-ebfc-45c9-a469-59388f320b7e" "1f98fff2-004d-4afa-9746-1dceb6a5cbe6")
-	)
-	(group "place:Debug: SWD, UART, reset, boot"
-		(members "098e87e8-775a-4317-ab6d-a252bd1943bc" "45a0fa4d-2b01-41e8-86ee-7137af7c5590"
-			"77c2969d-e58f-4558-b9ac-a95625df3670" "82b39b74-d08f-48f4-a54c-2d44e21537e1"
+	(group "place:USB-C iso in"
+		(members "164f89de-20dd-4124-8da1-ed733a12b481" "8bf929c0-e6ed-4a13-b934-a7add551427f"
+			"8fb93ad6-2053-4398-a265-31e07129cb04" "b78ded54-b343-4105-afc5-e6f0eb8666a2"
+			"c3da4db2-31b3-4f2b-b65c-7acc6d89cdcf"
 		)
 	)
-	(group "place:ADuM side 1 (PC)"
-		(members "013f1d01-8ae7-4bea-bddf-fd0585caa897" "4147e0b8-e13a-4cfc-b5f6-3a029c2d832c")
+	(group "place:ADuM side 2 (MCU)"
+		(members "03297722-b0ab-4e94-ac46-935e0d1636a3" "5789382e-05bf-4f47-ac0c-edcc57ff832b")
+	)
+	(group "place:B2B decoupling"
+		(members "19df6b39-ebfc-45c9-a469-59388f320b7e" "1f98fff2-004d-4afa-9746-1dceb6a5cbe6")
 	)
 	(group "place:LMR38010 3.3V"
@@
 		)
 	)
+	(group "place:B0505S out"
+		(members "284b26d2-9df1-4416-8676-dca69f693828" "a5682d17-5b93-43cc-8613-be2e1f29720d")
+	)
 	(group "place:STM32G474"
 		(members "07ca002f-af3b-4a0a-9ae5-d8a9b6ad320a" "0cf84e9a-2f72-4947-ac3b-132c75ace886"
@@
 		)
 	)
-	(group "place:B0505S out"
-		(members "284b26d2-9df1-4416-8676-dca69f693828" "a5682d17-5b93-43cc-8613-be2e1f29720d")
-	)
-	(group "place:ADuM side 2 (MCU)"
-		(members "03297722-b0ab-4e94-ac46-935e0d1636a3" "5789382e-05bf-4f47-ac0c-edcc57ff832b")
-	)
 	(group "place:+3V3A filter"
 		(members "0d43a9d1-6113-4fe9-be78-7558ef7dc3aa" "36a822bb-badb-4e42-8c95-392c8572b139"
@@
 		)
 	)
-	(group "place:USB-C iso in"
-		(members "164f89de-20dd-4124-8da1-ed733a12b481" "8bf929c0-e6ed-4a13-b934-a7add551427f"
-			"8fb93ad6-2053-4398-a265-31e07129cb04" "b78ded54-b343-4105-afc5-e6f0eb8666a2"
-			"c3da4db2-31b3-4f2b-b65c-7acc6d89cdcf"
+	(group "place:Debug: SWD, UART, reset, boot"
+		(members "098e87e8-775a-4317-ab6d-a252bd1943bc" "45a0fa4d-2b01-41e8-86ee-7137af7c5590"
+			"77c2969d-e58f-4558-b9ac-a95625df3670" "82b39b74-d08f-48f4-a54c-2d44e21537e1"
 		)
 	)
+	(group "place:ADuM side 1 (PC)"
+		(members "013f1d01-8ae7-4bea-bddf-fd0585caa897" "4147e0b8-e13a-4cfc-b5f6-3a029c2d832c")
+	)
 	(group "board_setup"
 		(locked yes)
@@
 	(group "floorplan"
 		(locked yes)
-		(members "001b429e-dd7c-4f40-8a24-234f29d0aeb9" "03e1abcb-1563-472f-b14c-51808568b32c"
-			"0f2637bf-7128-42e3-937a-57e743c3ad23" "1a9fe9b9-0de7-475f-87d4-dec7e5caef93"
-			"1de2d03f-4fa1-4118-8fe4-4f40ebbce767" "1e365e2b-0ec0-4ed5-b95a-998aa64b3470"
-			"20d8f301-e4c1-4a35-9761-4443ecb5c521" "29741cb1-dc90-45db-98c4-c791d7920c9e"
-			"29e75f12-f00c-4d1f-86e6-1c2476dad3a4" "3146e15a-c109-4cfd-a5aa-cf9d77e4757f"
-			"3cd1e70f-6f88-4ba3-9063-9896dfe2b369" "48ce6188-cabe-4df9-82ec-08ba38388382"
-			"49c6ab32-9e63-4cfd-afc3-2d65e0acbe51" "6ae665e8-bcfc-4819-8089-1741a9308f52"
-			"6b778096-8833-4273-af45-7750dda95f14" "808e6624-467d-449f-9f80-f00d81348fd3"
-			"819ffa4d-7945-447e-8f82-2e6b57d8e50f" "95550a94-a957-4f0d-9cd9-701bf8392e79"
-			"97522b60-311f-44c1-91e0-dbb4f9ea49d2" "9a331af8-f0dd-42d5-8cea-12d3387275bc"
-			"a281029b-7e2a-4351-9fd6-b7caf81232bb" "a39a56be-21ec-41b8-8bc3-94cbf5b99ef9"
-			"a5d934c9-499e-4121-a72c-551ce09cba60" "b0165ecf-90f5-4ba7-a3cc-672dabd8ca50"
-			"b1613d48-aae4-41db-b3fc-35f3267b3679" "bd1a0742-360a-4c96-a420-a175444cadb2"
-			"d7269c97-0abb-4ab1-ab17-26292f09418d" "dafe0343-02b1-4407-8a22-a6ff296d7903"
-			"ddb374b3-1b1d-4e9d-ada6-d8d70784c908" "de3c4a3e-bca6-4965-9491-8b4a3ca13ca9"
-			"de86cf41-a906-4bdb-a295-4a1518f1552b" "e4d6f45d-db3f-41e3-9fd5-c217b5be8e41"
-			"e7d9c251-0a59-4d1b-ad58-a6c0a06f7aa0" "e93cf797-6862-45f3-b10d-689b2deb0ba6"
-			"e9f0df60-c1f3-430f-a179-8b1115dbdc41" "ea595a76-e868-4f72-a512-6b1bc9c19d67"
-			"f7a408e9-214e-4747-88c5-8f928ac325ca"
+		(members "03e882ab-85ce-4f8f-8b1b-d5612879fa8b" "08866954-d14a-4343-a27e-05d163d09b0f"
+			"0d461552-9840-4d9c-92a1-420f420cacb2" "1a992d65-3574-411e-b372-0f1016af8d1c"
+			"1abe6c59-c7da-410a-bb61-08c105cb1b4d" "1c14cc4a-57e7-4e63-8e8d-baa59a9513f4"
+			"2f732be5-d1c2-4cf7-86c5-db43258706c4" "324fe440-7e0c-4b1d-83b7-b498eb4080a0"
+			"360e3a64-db5b-470b-aac1-4c56865afb11" "4c56c81a-7c43-4921-8d54-45f3c214948a"
+			"4fb5697e-63f3-44be-b536-4eadb5b873b0" "50b00232-0aef-47a2-b703-aa54ed3890f3"
+			"5ddc2ac7-bf50-4ed3-b015-85cf0768bb78" "6145c37f-9d30-4889-98ab-de28e17121b8"
+			"616f218c-48cf-47d3-8933-a3253cb8fd7c" "6897e889-04ec-44d5-a4e8-bd20c4d55984"
+			"7293084d-ecdd-45d9-81d9-8822920020dd" "7fa31b91-83dc-4a12-9110-9ca05ecfe23f"
+			"843fb230-58b3-4ead-9f79-a7878e336c4d" "8c8625f4-157b-4c7c-8f63-121526bebf31"
+			"9014324e-d30c-4699-adb6-1dbd02e66694" "9b321052-d620-44a6-94b2-b56e2890394d"
+			"ab852a35-d403-403b-be7d-62c8f09d60b8" "ad0e7f65-9073-496b-8e7e-13d33a58be2a"
+			"b04f2a54-6cfe-4a8e-aa84-ef711cedceb8" "bd3b83ab-2ab3-447a-8cdd-25720d188719"
+			"be1ddb42-fcd9-4183-aecc-650d3c5f1abe" "c22903a6-280a-4754-ad57-8ba6ebe85021"
+			"c9b3113f-535e-4ef1-9e3b-c3cc125aa95e" "c9e4b176-bc17-447b-92a7-6970e074ee83"
+			"cb97cc5e-d5ce-4901-9679-81df1a3f1a5c" "cbcd6627-8ee7-4cf1-92c0-a6e8bdf4eeb4"
+			"d329c1e7-1e39-451c-ac70-6d50afa45a4c" "dd644bb5-1fdb-4472-ab28-9891de850eca"
+			"edd9f1c1-2ea1-4f8e-a5d0-f164d3b322e2" "ee4fe7ce-f6b4-4239-9fb1-5b01e79ea34f"
+			"fd6f4de0-643a-447b-9be5-ed3ae500c5a4"
 		)
 	)
