File: kicad/supply_ui/supply_ui/supply_ui.kicad_pcb (KiCad board)
At the start: 2 copper layers, 73 parts, among them J1 to supply_control, J3 IPS 1.9in ST7789 SPI, J4 OE panel button, J5 POWER panel button, J6 OUTPUT panel button, Q1 2N7002, SW1 EC10E1220501, SW2 EC10E1220501, SW3 V WHEEL PUSH, SW4 I WHEEL PUSH, SW5 LEFT, SW6 RIGHT, SW7 ENTER, SW8 OUTPUT, SW9 POWER, U1 TCA9535PWR

Commit message: Checkpoint before ui routing
Parts:
- removed C11: 10n, Capacitor_SMD:C_0603_1608Metric
- removed D1: red, LED_SMD:LED_0805_2012Metric
- removed D2: green, LED_SMD:LED_0805_2012Metric
- removed H4: M3, MountingHole:MountingHole_3.2mm_M3
- removed J4: OE panel button, Connector_JST:JST_XH_B5B-XH-A_1x05_P2.50mm_Vertical
- removed J5: POWER panel button, Connector_JST:JST_XH_B2B-XH-A_1x02_P2.50mm_Vertical
- removed R21, R22: 330, Resistor_SMD:R_0603_1608Metric
- removed R25: 10k, Resistor_SMD:R_0603_1608Metric
- removed R26: 1k, Resistor_SMD:R_0603_1608Metric
- removed SW8: OUTPUT, Button_Switch_THT:SW_PUSH_6mm
- removed SW9: POWER, Button_Switch_THT:SW_PUSH_6mm
- BZ1, C1, C10, C12, C2, C3, C4, C5, C6, C7, C8, C9, D5, D6, J6, Q1, R1, R10, R11, R12, R15, R16, R17, R18, R19, R2, R20, R23, R24, R27, R28, R29, R3, R4, R5, R6, R7, R8, R9, TP1, TP2, TP3, TP4, TP7, TP8, TP9, U1: moved to B.Cu
- D3, D4: footprint LED_THT:LED_D3.0mm -> supply1:LED_D3.0mm_Standoff
- J1: footprint Connector_PinHeader_1.27mm:PinHeader_2x10_P1.27mm_Vertical -> Connector_PinHeader_2.54mm:PinHeader_2x10_P2.54mm_Horizontal; moved to B.Cu
- J3: value IPS 1.9in ST7789 SPI -> IPS 1.9in ST7789 SPI (wired); footprint Connector_PinSocket_2.54mm:PinSocket_1x08_P2.54mm_Vertical -> Connector_PinHeader_2.54mm:PinHeader_1x08_P2.54mm_Horizontal
- SW1, SW2: value EC10E1220501 -> EC10E1220505
- SW3, SW4, SW5, SW6, SW7: footprint Button_Switch_THT:SW_TH_Tactile_Omron_B3F-106x -> Button_Switch_THT:SW_TH_Tactile_Omron_B3F-102x
- moved C12 109.1 mm to (175.3, 67.4), turned to 90 degrees
- moved R29 95.2 mm to (169.8, 83.6), turned to 90 degrees
- moved TP9 87.5 mm to (166.3, 87.8)
- moved SW3 78.3 mm to (143.9, 122.2), turned to 90 degrees
- moved SW4 62.7 mm to (156.1, 115.8), turned to -90 degrees
- moved H1 58.4 mm to (180.0, 107.5)
- moved J6 56.0 mm to (128.5, 86.1), turned to 180 degrees
- moved D6 54.6 mm to (147.4, 69.2), turned to 90 degrees
- moved SW6 54.5 mm to (168.8, 96.8)
- moved C2 52.4 mm to (120.0, 79.7)
- moved U1 51.5 mm to (156.1, 83.7)
- moved SW7 50.3 mm to (153.8, 96.8)
- moved SW1 49.6 mm to (126.5, 119.0), turned to 90 degrees
- moved BZ1 48.0 mm to (156.8, 71.8), turned to 90 degrees
- moved R28 48.0 mm to (150.0, 63.9), turned to -90 degrees
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Routing:
- net +3V3: track 0.00 -> 2.28 mm
- net OE_LED_A: track 0.00 -> 0.52 mm
Other:
- board outline added: 70 x 72 mm
- board text added: "BOTTOM SIDE: connectors, expander, passives (under the display)"
- board text added: "supports 5 mm above it elsewhere; bottom side: wheels reach 1.4 mm, the on-off button 10 mm below"
- board text added: "top side: display module 9.7 mm above the board (y < -10.5), button sleeves and wheel"

Commit message: UI board routed
Parts:
- removed TP1, TP2, TP7, TP8, TP9: TestPoint, TestPoint:TestPoint_Pad_D1.0mm
- moved TP3 15.4 mm to (147.8, 90.9)
- moved D5 15.2 mm to (151.4, 76.2), turned to 90 degrees
- moved R20 15.1 mm to (149.2, 76.1), turned to 90 degrees
- moved TP4 11.7 mm to (147.8, 79.0)
- moved C9 7.50 mm to (156.0, 81.8), turned to 90 degrees
- moved U1 5.68 mm to (150.7, 85.6), turned to 90 degrees
- moved R27 3.09 mm to (125.9, 79.8), turned to -90 degrees
- moved R23 2.62 mm to (128.0, 79.8), turned to -90 degrees
- moved C8 2.31 mm to (155.8, 106.2)
- moved R24 0.91 mm to (129.7, 81.5), turned to -90 degrees
- moved R7 0.14 mm to (179.8, 116.4), turned to 180 degrees
- turned R1 to 0 degrees
- turned R3 to 0 degrees
Connections:
- U1 pad 18: N$8 -> (no net)
- U1 pad 19: N$9 -> (no net)
- U1 pad 20: N$10 -> (no net)
- U1 pad 7: N$1 (its old number) -> (no net)
- U1 pad 8: N$2 (its old number) -> (no net)
Routing:
- net +3V3: track 2.28 -> 349.7 mm, vias 0 -> 7
- net GND: track 0.33 -> 323.8 mm, vias 0 -> 6
- net ENC2_B: track 0.00 -> 107.1 mm, vias 0 -> 1
- net ENC2_A: track 0.00 -> 106.9 mm, vias 0 -> 2
- net ENC1_A: track 0.00 -> 75.7 mm
- net LCD_BL: track 0.00 -> 71.4 mm, vias 0 -> 1
- net ENC1_B: track 0.00 -> 67.6 mm
- net LED_CC_K: track 0.00 -> 65.2 mm, vias 0 -> 2
- net LED_CV_K: track 0.00 -> 62.1 mm, vias 0 -> 2
- net LCD_RST: track 0.00 -> 53.3 mm
- net LCD_CS: track 0.00 -> 46.2 mm
- net UI_INT: track 0.00 -> 46.0 mm, vias 0 -> 2
- net LCD_DC: track 0.00 -> 38.5 mm
- net LCD_MOSI: track 0.00 -> 37.1 mm
- net BUZZER: track 0.00 -> 36.4 mm, vias 0 -> 1
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- added copper zone on B.Cu, net GND
- added copper zone on F.Cu, net GND
Other:
- board text removed: "BOTTOM SIDE: connectors, expander, passives (under the display)"
- board text removed: "supports 5 mm above it elsewhere; bottom side: wheels reach 1.4 mm, the on-off button 10 mm below"
- board text removed: "top side: display module 9.7 mm above the board (y < -10.5), button sleeves and wheel"
